Commit message: Estevan's changes from 12-1-23

File: MovementModule/diffdrive_arduino/src/description/ros2_control/diffbot.ros2_control.xacro (robot description, xacro)
@@ -8,5 +8,4 @@
         <param name="right_wheel_name">right_wheel_joint</param>
         <param name="loop_rate">10</param>
-        <param name="baud_rate">115200</param>
       </hardware>
       <joint name="${prefix}left_wheel_joint">

File: RobotBringupModule/mws_robot/description/gazebo_control.xacro (robot description, xacro)
@@ -6,8 +6,8 @@
             <left_joint>left_wheel_joint</left_joint>
             <right_joint>right_wheel_joint</right_joint>
-            <wheel_separation>0.297</wheel_separation>
-            <wheel_diameter>0.066</wheel_diameter>
+            <wheel_separation>0.49</wheel_separation>
+            <wheel_diameter>0.0735</wheel_diameter>
             <!-- Limits -->
-            <max_wheel_torque>200</max_wheel_torque>
+            <max_wheel_torque>7</max_wheel_torque>
             <max_wheel_acceleration>10.0</max_wheel_acceleration>
             <!-- Output -->

File: RobotBringupModule/mws_robot/description/lidar.xacro (robot description, xacro)
@@ -1,30 +1,51 @@
 <?xml version="1.0"?>
 <robot xmlns:xacro="http://www.ros.org/wiki/xacro" >
+    <xacro:property name="laser_frame_offset_x" value="0.36"/>  <!-- Length and offset is specified in Meters -->
+    <xacro:property name="laser_frame_offset_z" value="1.253"/>
+    <xacro:property name="lidar_radius" value="0.05"/>
+    <xacro:property name="lidar_length" value="0.04"/>
+    <xacro:property name="lidar_mass" value="0.5"/>
+    <xacro:property name="lidar_cylinder_stand_radius" value="0.025"/>
+    <xacro:property name="lidar_cylinder_stand_length" value="0.3"/>
+    <xacro:property name="lidar_cylinder_stand_mass" value="1"/>
     <joint name="laser_joint" type="fixed">
         <parent link="chassis"/>
         <child link="laser_frame"/>
-        <origin xyz="0.122 0 0.212" rpy="0 0 0"/>
+        <origin xyz="${laser_frame_offset_x} 0 ${laser_frame_offset_z}" rpy="0 0 0"/>
     </joint>
     <link name="laser_frame">
+        <!-- LIDAR -->
         <visual>
+            <origin xyz="0 0 ${lidar_length / 2}"/>
             <geometry>
-                <cylinder radius="0.05" length="0.04"/>
-            </geometry>
-            <material name="black"/>
-        </visual>
-        <visual>
-            <origin xyz="0 0 -0.05"/>
-            <geometry>
-                <cylinder radius="0.01" length="0.1"/>
+                <cylinder radius="${lidar_radius}" length="${lidar_length}"/>
             </geometry>
             <material name="black"/>
         </visual>
         <collision>
+            <origin xyz="0 0 ${lidar_length / 2}"/>
             <geometry>
-                <cylinder radius="0.05" length="0.04"/>
+                <cylinder radius="${lidar_radius}" length="${lidar_length}"/>
             </geometry>
         </collision>
-        <xacro:inertial_cylinder mass="0.1" length="0.04" radius="0.05">
-            <origin xyz="0 0 0" rpy="0 0 0"/>
+        <xacro:inertial_cylinder mass="${lidar_mass}" length="${lidar_length}" radius="${lidar_radius}">
+            <origin xyz="0 0 ${lidar_length / 2}"/>
+        </xacro:inertial_cylinder>
+        <!-- LIDAR CYLINDER STAND -->
+        <visual>
+            <origin xyz="0 0 ${-lidar_cylinder_stand_length / 2}"/>
+            <geometry>
+                <cylinder radius="${lidar_cylinder_stand_radius}" length="${lidar_cylinder_stand_length}"/>
+            </geometry>
+            <material name="black"/>
+        </visual>
+        <collision>
+            <origin xyz="0 0 ${-lidar_cylinder_stand_length / 2}"/>
+            <geometry>
+                <cylinder radius="${lidar_cylinder_stand_radius}" length="${lidar_cylinder_stand_length}"/>
+            </geometry>
+        </collision>
+        <xacro:inertial_cylinder mass="${lidar_cylinder_stand_mass}" length="${lidar_cylinder_stand_length}" radius="${lidar_cylinder_stand_radius}">
+            <origin xyz="0 0 ${-lidar_cylinder_stand_length / 2}"/>
         </xacro:inertial_cylinder>
     </link>
@@ -33,5 +54,5 @@
         <sensor name="laser" type="ray">
             <pose> 0 0 0 0 0 0 </pose>
-            <visualize>false</visualize>
+            <visualize>true</visualize>
             <update_rate>10</update_rate>
             <ray>

File: RobotBringupModule/mws_robot/description/mws_robot.ros2_control.xacro (robot description, xacro)
@@ -1,4 +1,5 @@
 <?xml version="1.0"?>
 <robot xmlns:xacro="http://www.ros.org/wiki/xacro">
+  <xacro:unless value="$(arg sim_mode)">
     <ros2_control name="diffbot" type="system">
       <hardware>
@@ -19,3 +20,33 @@
       </joint>
     </ros2_control>
+  </xacro:unless>
+  <xacro:if value="$(arg sim_mode)">
+    <ros2_control name="GazeboSystem" type="system">
+        <hardware>
+            <plugin>gazebo_ros2_control/GazeboSystem</plugin>
+        </hardware>
+        <joint name="left_wheel_joint">
+            <command_interface name="velocity">
+                <param name="min">-10</param>
+                <param name="max">10</param>
+            </command_interface>
+            <state_interface name="velocity"/>
+            <state_interface name="position"/>
+        </joint>
+        <joint name="right_wheel_joint">
+            <command_interface name="velocity">
+                <param name="min">-10</param>
+                <param name="max">10</param>
+            </command_interface>
+            <state_interface name="velocity"/>
+            <state_interface name="position"/>
+        </joint>
+    </ros2_control>
+  </xacro:if>
+  <gazebo>
+    <plugin name="gazebo_ros2_control" filename="libgazebo_ros2_control.so">
+        <parameters>$(find mws_robot)/params/diffbot_controllers.yaml</parameters>
+        <parameters>$(find mws_robot)/params/ros2_sim_time.yaml</parameters>
+    </plugin>
+</gazebo>
 </robot>

File: RobotBringupModule/mws_robot/description/mws_robot_core.xacro (robot description, xacro)
@@ -1,18 +1,21 @@
 <?xml version="1.0"?>
 <robot xmlns:xacro="http://www.ros.org/wiki/xacro" >
-    <xacro:property name="chassis_length" value="0.335"/>
-    <xacro:property name="chassis_width" value="0.265"/>
-    <xacro:property name="chassis_height" value="0.138"/>
-    <xacro:property name="chassis_mass" value="1.0"/>
-    <xacro:property name="wheel_radius" value="0.033"/>
-    <xacro:property name="wheel_thickness" value="0.026"/>
-    <xacro:property name="wheel_mass" value="0.05"/>
+    <xacro:property name="chassis_length" value="0.72"/>  <!-- Length and offset is specified in Meters -->
+    <xacro:property name="chassis_width" value="0.71"/>
+    <xacro:property name="chassis_height" value="0.955"/>
+    <xacro:property name="chassis_offset_z" value="0.105"/>
+    <xacro:property name="chassis_offset_x" value="0.205"/>
+    <xacro:property name="chassis_mass" value="30.0"/>  <!-- Mass is specified in Kilograms -->
+    <xacro:property name="wheel_radius" value="0.0735"/>
+    <xacro:property name="wheel_thickness" value="0.03"/>
+    <xacro:property name="wheel_mass" value="1.5"/>
     <xacro:property name="wheel_offset_x" value="0.226"/>
-    <xacro:property name="wheel_offset_y" value="0.1485"/>
-    <xacro:property name="wheel_offset_z" value="0.01"/>
-    <xacro:property name="caster_wheel_radius" value="0.01"/>
-    <xacro:property name="caster_wheel_mass" value="0.01"/>
-    <xacro:property name="caster_wheel_offset_x" value="0.075"/>
-    <xacro:property name="caster_wheel_offset_z" value="${wheel_offset_z - wheel_radius + caster_wheel_radius}"/>
+    <xacro:property name="wheel_offset_y" value="0.245"/>
+    <xacro:property name="wheel_offset_z" value="${wheel_radius}"/>
+    <xacro:property name="caster_wheel_radius" value="${chassis_offset_z / 2}"/>
+    <xacro:property name="caster_wheel_mass" value="1"/>
+    <xacro:property name="caster_wheel_offset_x" value="0.57"/>
+    <xacro:property name="caster_wheel_offset_y" value="0.22"/>
+    <xacro:property name="caster_wheel_offset_z" value="${-chassis_offset_z / 2}"/>
     <!-- BASE LINK -->
     <link name="base_link">
@@ -30,5 +33,5 @@
         <parent link="base_link"/>
         <child link="chassis"/>
-        <origin xyz="${-wheel_offset_x} 0 ${-wheel_offset_z}"/>
+        <origin xyz="${-chassis_offset_x} 0 ${chassis_offset_z}"/>
     </joint>
     <link name="chassis">
@@ -46,5 +49,5 @@
             </geometry>
         </collision>
-        <xacro:inertial_box mass="0.5" x="${chassis_length}" y="${chassis_width}" z="${chassis_height}">
+        <xacro:inertial_box mass="${chassis_mass}" x="${chassis_length}" y="${chassis_width}" z="${chassis_height}">
             <origin xyz="${chassis_length/2} 0 ${chassis_height/2}" rpy="0 0 0"/>
         </xacro:inertial_box>
@@ -57,5 +60,5 @@
         <parent link="base_link"/>
         <child link="left_wheel"/>
-        <origin xyz="0 ${wheel_offset_y} 0" rpy="-${pi/2} 0 0" />
+        <origin xyz="0 ${wheel_offset_y} ${wheel_offset_z}" rpy="-${pi/2} 0 0" />
         <axis xyz="0 0 1"/>
     </joint>
@@ -83,5 +86,5 @@
         <parent link="base_link"/>
         <child link="right_wheel"/>
-        <origin xyz="0 ${-wheel_offset_y} 0" rpy="${pi/2} 0 0" />
+        <origin xyz="0 ${-wheel_offset_y} ${wheel_offset_z}" rpy="${pi/2} 0 0" />
         <axis xyz="0 0 -1"/>
     </joint>
@@ -105,11 +108,11 @@
         <material>Gazebo/Blue</material>
     </gazebo>
-    <!-- CASTER WHEEL LINK -->
-    <joint name="caster_wheel_joint" type="fixed">
+    <!-- LEFT CASTER WHEEL LINK -->
+    <joint name="left_caster_wheel_joint" type="fixed">
         <parent link="chassis"/>
-        <child link="caster_wheel"/>
-        <origin xyz="${caster_wheel_offset_x} 0 ${caster_wheel_offset_z}"/>
+        <child link="left_caster_wheel"/>
+        <origin xyz="${caster_wheel_offset_x} ${caster_wheel_offset_y} ${caster_wheel_offset_z}"/>
     </joint>
-    <link name="caster_wheel">
+    <link name="left_caster_wheel">
         <visual>
             <geometry>
@@ -127,5 +130,32 @@
         </xacro:inertial_sphere>
     </link>
-    <gazebo reference="caster_wheel">
+    <gazebo reference="left_caster_wheel">
+        <material>Gazebo/White</material>
+        <mu1 value="0.001"/>
+        <mu2 value="0.001"/>
+    </gazebo>
+    <!-- RIGHT CASTER WHEEL LINK -->
+    <joint name="right_caster_wheel_joint" type="fixed">
+        <parent link="chassis"/>
+        <child link="right_caster_wheel"/>
+        <origin xyz="${caster_wheel_offset_x} ${-caster_wheel_offset_y} ${caster_wheel_offset_z}"/>
+    </joint>
+    <link name="right_caster_wheel">
+        <visual>
+            <geometry>
+                <sphere radius="${caster_wheel_radius}"/>
+            </geometry>
+            <material name="white"/>
+        </visual>
+        <collision>
+            <geometry>
+                <sphere radius="${caster_wheel_radius}"/>
+            </geometry>
+        </collision>
+        <xacro:inertial_sphere mass="${caster_wheel_mass}" radius="${caster_wheel_radius}">
+            <origin xyz="0 0 0" rpy="0 0 0"/>
+        </xacro:inertial_sphere>
+    </link>
+    <gazebo reference="right_caster_wheel">
         <material>Gazebo/White</material>
         <mu1 value="0.001"/>
